File: kicad_diseño/fuente_simetrica_24v/control.kicad_sch (KiCad schematic)
At the start: 0 parts

Commit message: Update Fte - Control.
Parts:
- added J4: Conn_01x04_Socket, symbol Connector:Conn_01x04_Socket
- added R12: 10k, symbol Device:R
- added SW1, SW2: SW_Push, symbol Switch:SW_Push
- added U6: ESP32-WROOM-32E, RF_Module:ESP32-WROOM-32D, symbol RF_Module:ESP32-WROOM-32E
- added U7: AMS1117-3.3, Package_TO_SOT_SMD:SOT-223-3_TabPin2, symbol Regulator_Linear:AMS1117-3.3
Connections:
- new net: SW1.1, U6.25 (IO0)
- new net: R12.2, SW2.2, U6.3 (EN)
- new net +3.3V: J4.1 (Pin_1), R12.1, U6.2 (VDD), U7.2 (VO)
- new net +5V: U7.3 (VI)
- new net GND: J4.4 (Pin_4), SW1.2, SW2.1, U6.1 (GND), U6.15 (GND), U6.38 (GND), U6.39 (GND), U7.1 (GND)
- new net IO12: U6.14 (IO12)
- new net IO13: U6.16 (IO13)
- new net IO14: U6.13 (IO14)
- new net IO15: U6.23 (IO15)
- new net IO16: U6.27 (IO16)
- new net IO17: U6.28 (IO17)
- new net IO18: U6.30 (IO18)
- new net IO19: U6.31 (IO19)
- new net IO2: U6.24 (IO2)
- new net IO21: U6.33 (IO21)
- new net IO22: U6.36 (IO22)
- new net IO23: U6.37 (IO23)
- new net IO25: U6.10 (IO25)
- new net IO26: U6.11 (IO26)
- new net IO27: U6.12 (IO27)
- new net IO32: U6.8 (IO32)
- new net IO33: U6.9 (IO33)
- new net IO34: U6.6 (IO34)
- new net IO35: U6.7 (IO35)
- new net IO4: U6.26 (IO4)
- new net IO5: U6.29 (IO5)
- new net RX: J4.3 (Pin_3), U6.34 (RXD0/IO3)
- new net TX: J4.2 (Pin_2), U6.35 (TXD0/IO1)
- no-connect marks 0 -> 2

Commit message: Update Fte - Pcb
Parts:
- added BZ1: Buzzer, symbol Device:Buzzer
- added D12, D13, D14: D_Zener, symbol Device:D_Zener
- added DS1: WC1602A, Display:WC1602A, symbol Display_Character:WC1602A
- added Q3: BC548, Package_TO_SOT_THT:TO-92_Inline, symbol Transistor_BJT:BC548
- added R13, R14, R15, R16, R17, R18, R8: R, symbol Device:R
- added RV2, RV5: R_Potentiometer_Trim, symbol Device:R_Potentiometer_Trim
- added RV4: 10k, symbol Device:R_Potentiometer_Trim
- added U10, U8: LM358, symbol Amplifier_Operational:LM358
Connections:
- net IO13 is gone; now on net RELE_POSITIVO: U6.16 (IO13)
- net +5V: now also DS1.15 (LED(+)), DS1.2 (VDD), Q3.1 (C), RV4.1, U10.8 (V+), U8.8 (V+)
- net GND: now also BZ1.2 (-), D12.2 (A), D13.2 (A), D14.2 (A), DS1.1 (VSS), DS1.16 (LED(-)), DS1.5 (R/W), R8.2, RV2.2, RV2.3, RV4.3, RV5.2, RV5.3, U10.3 (+)
- net IO14: now also R15.1
- net IO15: now also D12.1 (K), U8.1, U8.2 (-)
- net IO17: now also DS1.6 (E)
- net IO18: now also DS1.4 (RS)
- net IO19: now also DS1.7 (D0)
- net IO21: now also DS1.8 (D1)
- net IO22: now also DS1.9 (D2)
- net IO23: now also DS1.10 (D3)
- net IO34: now also D13.1 (K), R14.2, U8.7
- net IO35: now also D14.1 (K), R17.2, U10.1
- net IO12 renamed RELE_POSITIVO
- new net: R14.1, R8.1, U8.6 (-)
- new net: R16.1, R18.2, RV5.1
- new net: R13.2, RV2.1, U8.3 (+)
- new net: Q3.2 (B), R15.2
- new net: R16.2, R17.1, U10.2 (-)
- new net: BZ1.1 (+), Q3.3 (E)
- new net: DS1.3 (VO), RV4.2
- new net +VDC: R13.1
- new net -5V: U10.4 (V-), U8.4 (V-)
- new net -VDC: R18.1
- new net Vshunt: U8.5 (+)
- no-connect marks 2 -> 6

Commit message: Update Fte - Pcb
Parts:
- added C13, C14: C, Capacitor_THT:C_Disc_D5.0mm_W2.5mm_P2.50mm, symbol Device:C
- added R19, R6, R9: 10k, Resistor_THT:R_Axial_DIN0207_L6.3mm_D2.5mm_P10.16mm_Horizontal, symbol Device:R
- added SW3: RotaryEncoder_Switch, Connector_PinSocket_2.54mm:PinSocket_1x04_P2.54mm_Vertical, symbol Device:RotaryEncoder_Switch
- BZ1: footprint (none) -> Buzzer_Beeper:MagneticBuzzer_ProSignal_ABI-009-RC
- D12, D13, D14: footprint (none) -> Diode_THT:D_5W_P12.70mm_Horizontal
- J4: footprint (none) -> Connector_PinSocket_2.54mm:PinSocket_1x04_P2.54mm_Vertical
- R12, R13, R14, R15, R16, R17, R8: footprint (none) -> Resistor_THT:R_Axial_DIN0207_L6.3mm_D2.5mm_P10.16mm_Horizontal
- R18: footprint (none) -> LED_THT:LED_D5.0mm
- RV2, RV5: footprint (none) -> Potentiometer_THT:Potentiometer_Bourns_3296W_Vertical
- RV4: footprint (none) -> Connector_PinHeader_2.54mm:PinHeader_1x03_P2.54mm_Vertical
- SW1, SW2: footprint (none) -> Button_Switch_THT:SW_PUSH_6mm
- U10, U8: footprint (none) -> Package_DIP:DIP-8_W7.62mm_LongPads
Connections:
- net +3.3V: now also R19.1, R6.1, R9.1
- net GND: now also C13.2, C14.2, SW3.S2
- net IO2: now also R19.2, SW3.S1
- net IO25: now also C13.1, R6.2, SW3.A
- net IO26: now also C14.1, R9.2, SW3.B
Other:
- moved on the sheet: BZ1, Q3, R15

Commit message: Update Fte - Pcb
Parts:
- D12, D13, D14: footprint Diode_THT:D_5W_P12.70mm_Horizontal -> Diode_THT:D_DO-35_SOD27_P7.62mm_Horizontal
- Q3: footprint Package_TO_SOT_THT:TO-92_Inline -> Package_TO_SOT_THT:TO-92_Inline_Wide
- SW3: footprint Connector_PinSocket_2.54mm:PinSocket_1x04_P2.54mm_Vertical -> Rotary_Encoder:RotaryEncoder_Alps_EC11E-Switch_Vertical_H20mm
Connections:
- net GND: now also SW3.C
Changed lines of the file:
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@@
 	(wire
 		(pts
+			(xy 119.38 181.61) (xy 120.65 181.61)
+		)
+		(stroke
+			(width 0)
+			(type default)
+		)
+	)
+	(wire
+		(pts
 			(xy 73.66 35.56) (xy 76.2 35.56)
 		)
@@
 	(wire
 		(pts
+			(xy 119.38 184.15) (xy 119.38 181.61)
+		)
+		(stroke
+			(width 0)
+			(type default)
+		)
+	)
+	(wire
+		(pts
 			(xy 151.13 68.58) (xy 151.13 69.85)
 		)
@@
 	(wire
 		(pts
+			(xy 120.65 181.61) (xy 120.65 176.53)
+		)
+		(stroke
+			(width 0)
+			(type default)
+		)
+	)
+	(wire
+		(pts
 			(xy 29.21 33.02) (xy 29.21 35.56)
 		)
@@
 	(wire
 		(pts
+			(xy 120.65 176.53) (xy 121.92 176.53)
+		)
+		(stroke
+			(width 0)
+			(type default)
+		)
+	)
+	(wire
+		(pts
 			(xy 151.13 59.69) (xy 151.13 60.96)
 		)
@@
 			)
 		)
-		(property "Footprint" "Connector_PinSocket_2.54mm:PinSocket_1x04_P2.54mm_Vertical"
+		(property "Footprint" "Rotary_Encoder:RotaryEncoder_Alps_EC11E-Switch_Vertical_H20mm"
 			(at 125.73 172.466 0)
 			(effects
@@
 			)
 		)
-		(property "Footprint" "Diode_THT:D_5W_P12.70mm_Horizontal"
+		(property "Footprint" "Diode_THT:D_DO-35_SOD27_P7.62mm_Horizontal"
 			(at 203.2 144.78 0)
 			(effects
@@
 			)
 		)
-		(property "Footprint" "Package_TO_SOT_THT:TO-92_Inline"
+		(property "Footprint" "Package_TO_SOT_THT:TO-92_Inline_Wide"
 			(at 116.84 135.255 0)
 			(effects
@@
 			)
 		)
-		(property "Footprint" "Diode_THT:D_5W_P12.70mm_Horizontal"
+		(property "Footprint" "Diode_THT:D_DO-35_SOD27_P7.62mm_Horizontal"
 			(at 205.74 77.47 0)
 			(effects
@@
 			)
 		)
-		(property "Footprint" "Diode_THT:D_5W_P12.70mm_Horizontal"
+		(property "Footprint" "Diode_THT:D_DO-35_SOD27_P7.62mm_Horizontal"
 			(at 205.74 99.06 0)
 			(effects
@@
 					(unit 1)
 				)
+			)
+		)
+	)
+	(symbol
+		(lib_id "power:GND")
+		(at 119.38 184.15 0)
+		(unit 1)
+		(exclude_from_sim no)
+		(in_bom yes)
+		(on_board yes)
+		(dnp no)
+		(fields_autoplaced yes)
+		(property "Reference" "#PWR057"
+			(at 119.38 190.5 0)
+			(effects
+				(font
+					(size 1.27 1.27)
+				)
+				(hide yes)
+			)
+		)
+		(property "Value" "GND"
+			(at 119.38 189.23 0)
+			(effects
+				(font
+					(size 1.27 1.27)
+				)
+			)
+		)
+		(property "Footprint" ""
+			(at 119.38 184.15 0)
+			(effects
+				(font
+					(size 1.27 1.27)
+				)
+				(hide yes)
+			)
+		)
+		(property "Datasheet" ""
+			(at 119.38 184.15 0)
+			(effects
+				(font
+					(size 1.27 1.27)
+				)
+				(hide yes)
+			)
+		)
+		(property "Description" "Power symbol creates a global label with name \"GND\" , ground"
+			(at 119.38 184.15 0)
+			(effects
+				(font
+					(size 1.27 1.27)
+				)
+				(hide yes)
+			)
+		)
+		(pin "1"
+		)
+		(instances
+			(project "fuente_simetrica_24v"
+				(path "/36af1dc6-a136-49f2-a170-bbda6635ecf8/2e9e32ce-e371-4542-a5d5-48143618db0b"
+					(reference "#PWR057")
+					(unit 1)
+				)

Commit message: Update Fte
Parts:
- R18: footprint LED_THT:LED_D5.0mm -> Resistor_THT:R_Axial_DIN0207_L6.3mm_D2.5mm_P10.16mm_Horizontal
- RV4: footprint Connector_PinHeader_2.54mm:PinHeader_1x03_P2.54mm_Vertical -> Potentiometer_THT:Potentiometer_Bourns_3296W_Vertical
- SW1: value SW_Push -> BOOT
- SW2: value SW_Push -> RESET
Other:
- note added: "Alimentación"
- note added: "ESP32"
- note added: "LCD 16X2"
- moved on the sheet: DS1, R12, RV4, SW1, SW2, U6, U7
