File: kicad_diseño/fuente_simetrica_24v/control.kicad_sch (KiCad schematic)
At the start: 37 parts, among them J4 Comunicacion, J7 Conn_02x03_Odd_Even, J8 Conn_02x03_Odd_Even, Q3 BC548, SW1 BOOT, SW2 RESET, SW3 RotaryEncoder_Switch, U10 LM358, U11 LM324, U6 ESP32-WROOM-32E, U7 AMS1117-3.3

Commit message: Update Fte - Control
Parts:
- J7, J8: footprint Connector_IDC:IDC-Header_2x03_P2.54mm_Horizontal -> Connector_PinSocket_2.54mm:PinSocket_2x03_P2.54mm_Horizontal
Changed lines of the file:
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@@
 			)
 		)
-		(property "Footprint" "Connector_IDC:IDC-Header_2x03_P2.54mm_Horizontal"
+		(property "Footprint" "Connector_PinSocket_2.54mm:PinSocket_2x03_P2.54mm_Horizontal"
 			(at 189.23 29.21 0)
 			(effects
@@
 			)
 		)
-		(property "Footprint" "Connector_IDC:IDC-Header_2x03_P2.54mm_Horizontal"
+		(property "Footprint" "Connector_PinSocket_2.54mm:PinSocket_2x03_P2.54mm_Horizontal"
 			(at 226.06 29.21 0)
 			(effects
