File: kicad_diseño/fuente_simetrica_24v/control.kicad_sch (KiCad schematic)
At the start: 32 parts, among them J4 Comunicacion, J7 Conn_02x03_Odd_Even, J8 Conn_02x03_Odd_Even, Q3 BC548, SW1 BOOT, SW2 RESET, SW3 RotaryEncoder_Switch, U10 LM358, U6 ESP32-WROOM-32E, U7 AMS1117-3.3, U8 TL082

Commit message: Update Fte - Diseño pcb
Parts:
- R8: footprint (none) -> Resistor_THT:R_Axial_DIN0207_L6.3mm_D2.5mm_P10.16mm_Horizontal
- RV2: footprint (none) -> Potentiometer_THT:Potentiometer_Bourns_3296W_Vertical
- U8: footprint (none) -> Package_DIP:DIP-8_W7.62mm_LongPads
Connections:
- net V2_shunt: no longer names the net of J8.3 (Pin_3)
- no-connect marks 6 -> 7
Other:
- note added: "(-3.3)V - 0V"
- note added: "0V - 3.3V"
- note removed: "G = 1 + 50k/RG"
- moved on the sheet: R18, RV5, U10A
