File: kicad_diseño/fuente_simetrica_24v/alimentacion.kicad_sch (KiCad schematic)
At the start: 22 parts, among them J1 Entrada +-24V, U1 LM317_TO-220, U2 LM337_TO220, U3 LM7805_TO220

Commit message: Update Fte - Control.
Parts:
- added D10, D11, D8: LED, symbol Device:LED
- added D7, D9: 1N4007, Diode_THT:D_DO-41_SOD81_P10.16mm_Horizontal, symbol Diode:1N4007
- added J2: 5V_salida, symbol Connector:Screw_Terminal_01x02
- added J3: Screw_Terminal_01x03, symbol Connector:Screw_Terminal_01x03
- added K1, K2: SANYOU_SRD_Form_C, Relay_THT:Relay_SPDT_SANYOU_SRD_Series_Form_C, symbol Relay:SANYOU_SRD_Form_C
- added Q1, Q2: BC548, Package_TO_SOT_THT:TO-92_Inline, symbol Transistor_BJT:BC548
- added R10, R11, R4, R5: R, symbol Device:R
- added R3: 120, symbol Device:R
- added R6, R9: r_led, symbol Device:R
- added R7, R8: shunt, symbol Device:R
- added RV1: 10k, symbol Device:R_Potentiometer
- added U4, U5: PC817, Package_DIP:DIP-4_W7.62mm, symbol Isolator:PC817
- C3, C4: value 1200uF -> 2000uF
- R2: value R -> 120
Connections:
- net GND: now also C7.2, C8.2, U3.2 (GND), D8.1 (K), J2.2 (Pin_2), J3.2 (Pin_2), Q1.3 (E), Q2.3 (E), R10.2, R11.2, R6.2, R9.2, RV1.1
- net +5V: now reaches C8.1, D4.2 (A), U3.3 (VO)
- net +5V: now also D7.1 (K), D9.1 (K), J2.1 (Pin_1), K1.5, K2.5, R3.1, U4.4, U5.4
- net +VDC: now reaches C2.1, D2.2 (A), D5.1 (K), R1.1, U1.2 (VO)
- net +VDC: now also K1.1
- net -VDC: now reaches C6.2, D3.1 (K), D6.2 (A), R2.2, U2.3 (VO)
- net -VDC: now also K2.1
- net PWM2: no longer names the net of R2.1, U2.1 (ADJ)
- net PWM2: now also RV1.2, RV1.3
- new net: D10.1 (K), R6.1
- new net: D10.2 (A), K1.4
- new net: D9.2 (A), K2.2, Q2.1 (C)
- new net: Q2.2 (B), R5.2
- new net: J3.1 (Pin_1), R7.2
- new net: J3.3 (Pin_3), R8.2
- new net: D7.2 (A), K1.2, Q1.1 (C)
- new net: K1.3, R7.1
- new net: D8.2 (A), R3.2
- new net: R11.1, U5.2
- new net: R10.1, U4.2
- new net: R4.1, U4.3
- new net: D11.1 (K), R9.1
- new net: D11.2 (A), K2.4
- new net: K2.3, R8.1
- new net: Q1.2 (B), R4.2
- new net: R5.1, U5.3
- new net RELE_NEGATIVO: U5.1
- new net RELE_POSITIVO: U4.1
Other:
- moved on the sheet: C9, D5

Commit message: Update Fte - Pcb
Parts:
- removed R8: shunt, symbol Device:R
- added C11: 2.2uF, symbol Device:C_Polarized_US
- added C12: 1uF, symbol Device:C_Polarized_US
- added RV3: 10k, symbol Device:R_Potentiometer
- added U9: LM7905_TO220, Package_TO_SOT_THT:TO-220-3_Vertical, symbol Regulator_Linear:LM7905_TO220
Connections:
- net GND: now also R7.1, C11.1, C12.1, RV3.3, U9.1 (GND); no longer J3.2 (Pin_2)
- net at C4.2, C5.2, D1.3 (-)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: now also C11.2, U9.2 (VI)
- net at J3.1 (Pin_1): now also K1.3; no longer R7.2
- net at J3.3 (Pin_3): now also K2.3
- net PWM1: no longer names the net of R1.2, U1.1 (ADJ)
- net PWM1: now also RV3.1, RV3.2
- new net -5V: C12.2, U9.3 (VO)
- new net Vshunt: J3.2 (Pin_2), R7.2
Other:
- moved on the sheet: R1, R7

Commit message: Update Fte - Pcb
Parts:
- removed D10, D11: LED, symbol Device:LED
- removed R6, R9: r_led, symbol Device:R
- C1, C11, C12, C2, C5, C8: footprint (none) -> Capacitor_THT:CP_Radial_D4.0mm_P1.50mm
- C10, C6, C7, C9: footprint (none) -> Capacitor_THT:CP_Radial_D4.0mm_P2.00mm
- C3, C4: footprint (none) -> Capacitor_THT:CP_Radial_D14.0mm_P5.00mm
- D8: footprint (none) -> LED_THT:LED_D5.0mm
- J1: footprint (none) -> TerminalBlock:TerminalBlock_bornier-3_P5.08mm
- J2: footprint (none) -> TerminalBlock:TerminalBlock_bornier-2_P5.08mm
- J3: footprint (none) -> Diode_THT:D_5W_P12.70mm_Horizontal
- R1, R10, R11, R2, R3, R4, R5, R7: footprint (none) -> Resistor_THT:R_Axial_DIN0207_L6.3mm_D2.5mm_P10.16mm_Horizontal
- RV1, RV3: footprint (none) -> Connector_PinHeader_2.54mm:PinHeader_1x03_P2.54mm_Vertical
Connections:
- no-connect marks 0 -> 2

Commit message: Update Fte - Pcb
Parts:
- J3: footprint Diode_THT:D_5W_P12.70mm_Horizontal -> TerminalBlock:TerminalBlock_bornier-3_P5.08mm
- Q1, Q2: footprint Package_TO_SOT_THT:TO-92_Inline -> Package_TO_SOT_THT:TO-92_Inline_Wide
Changed lines of the file:
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@@
 			)
 		)
-		(property "Footprint" "Package_TO_SOT_THT:TO-92_Inline"
+		(property "Footprint" "Package_TO_SOT_THT:TO-92_Inline_Wide"
 			(at 74.93 179.705 0)
 			(effects
@@
 			)
 		)
-		(property "Footprint" "Diode_THT:D_5W_P12.70mm_Horizontal"
+		(property "Footprint" "TerminalBlock:TerminalBlock_bornier-3_P5.08mm"
 			(at 124.46 121.92 0)
 			(effects
@@
 			)
 		)
-		(property "Footprint" "Package_TO_SOT_THT:TO-92_Inline"
+		(property "Footprint" "Package_TO_SOT_THT:TO-92_Inline_Wide"
 			(at 74.93 128.905 0)
 			(effects

Commit message: Update Fte
Parts:
- added J5, J6: Conn_02x03_Odd_Even, symbol Connector_Generic:Conn_02x03_Odd_Even
- J3: value Screw_Terminal_01x03 -> Salida +-24V
- RV3: footprint Connector_PinHeader_2.54mm:PinHeader_1x03_P2.54mm_Vertical -> Connector_PinSocket_2.54mm:PinSocket_1x03_P2.54mm_Vertical
Connections:
- net +5V: now also J6.1 (Pin_1)
- net +VDC: now also J5.2 (Pin_2)
- net -5V: now also J6.3 (Pin_3)
- net -VDC: now also J5.4 (Pin_4)
- net GND: now also J5.3 (Pin_3), J5.5 (Pin_5), J5.6 (Pin_6), J6.5 (Pin_5), J6.6 (Pin_6)
- net RELE_NEGATIVO renamed RELE 2
- net RELE 2: now also J6.4 (Pin_4)
- net RELE_POSITIVO renamed RELE 1
- net RELE 1: now also J6.2 (Pin_2)
- net Vshunt renamed V1_shunt
- net V1_shunt: now also J5.1 (Pin_1)
Other:
- note added: "Alimentación Salida: +- 24V +- 5V"
- note added: "Conectores"
- note added: "Salida de +-24V"
- company: (none) -> Zuliani, Agustín
- title: (none) -> Circuito de potencia
- moved on the sheet: C1, C10, C11, C12, C2, C3, C4, C5, C6, C7, C8, C9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

Commit message: Update Fte
Parts:
- added TP1, TP4: lm337_out, TestPoint:TestPoint_2Pads_Pitch5.08mm_Drill1.3mm, symbol Connector:TestPoint_2Pole
- added TP2: lm7805_out, TestPoint:TestPoint_2Pads_Pitch5.08mm_Drill1.3mm, symbol Connector:TestPoint_2Pole
- added TP3: lm7905_out, TestPoint:TestPoint_2Pads_Pitch5.08mm_Drill1.3mm, symbol Connector:TestPoint_2Pole
- C3, C4: value 2000uF -> 2200uF
- J5, J6: footprint (none) -> Connector_IDC:IDC-Header_2x03_P2.54mm_Horizontal
- RV1: value 10k -> 5k
- RV3: value 10k -> 5k; footprint Connector_PinSocket_2.54mm:PinSocket_1x03_P2.54mm_Vertical -> Connector_PinHeader_2.54mm:PinHeader_1x03_P2.54mm_Vertical
Connections:
- net +5V: now also J5.1 (Pin_1), TP2.1; no longer J6.1 (Pin_1)
- net +VDC: now also TP1.1
- net -5V: now also J5.3 (Pin_3), TP3.1; no longer J6.3 (Pin_3)
- net -VDC: now also TP4.1
- net GND: now also J6.3 (Pin_3), TP1.2, TP2.2, TP3.2, TP4.2; no longer J5.3 (Pin_3)
- net V1_shunt: now also J6.1 (Pin_1); no longer J5.1 (Pin_1)
- net lm317_vi: now reaches C1.1, C3.1, C7.1, D1.1 (+), D2.1 (K), D4.1 (K), U1.3 (VI), U3.1 (VI)
- net lm317_vadj: now reaches R1.2, RV3.1, RV3.2, U1.1 (ADJ)
- net lm317_vadj: now also C9.1, D5.2 (A)
- net lm337_vadj: now reaches R2.1, RV1.2, RV1.3, U2.1 (ADJ)
- net lm337_vadj: now also C10.2, D6.1 (K)
- net lm337_vi: now reaches C11.2, C4.2, C5.2, D1.3 (-), D3.2 (A), U2.2 (VI), U9.2 (VI)
- net puente_in: now reaches D1.4, J1.1 (Pin_1)
- net puente_in2: now reaches D1.2, J1.3 (Pin_3)
- net rele 1: now reaches J3.1 (Pin_1), K1.3
- net rele 2: now reaches J3.3 (Pin_3), K2.3
Other:
- moved on the sheet: D5, J5, J6

Commit message: Update Fte - Fte Potencia
Parts:
- removed D1: W01G, Diode_THT:Diode_Bridge_Round_D9.8mm, symbol Diode_Bridge:W01G
- removed TP1, TP4: lm337_out, TestPoint:TestPoint_2Pads_Pitch5.08mm_Drill1.3mm, symbol Connector:TestPoint_2Pole
- removed TP2: lm7805_out, TestPoint:TestPoint_2Pads_Pitch5.08mm_Drill1.3mm, symbol Connector:TestPoint_2Pole
- removed TP3: lm7905_out, TestPoint:TestPoint_2Pads_Pitch5.08mm_Drill1.3mm, symbol Connector:TestPoint_2Pole
- added D1, D13, D15, D16: 1N5407, Diode_THT:D_DO-201AD_P15.24mm_Horizontal, symbol Diode:1N5407
- added TP1: lm337_out, TestPoint:TestPoint_Pad_D3.0mm, symbol Connector:TestPoint
- added TP2: lm317_out, TestPoint:TestPoint_Pad_D3.0mm, symbol Connector:TestPoint
- added TP3: lm7905_out, TestPoint:TestPoint_Pad_D3.0mm, symbol Connector:TestPoint
- added TP5: lm7805_out, TestPoint:TestPoint_Pad_D3.0mm, symbol Connector:TestPoint
- C1, C11, C12, C2, C5, C8: footprint Capacitor_THT:CP_Radial_D4.0mm_P1.50mm -> Capacitor_THT:CP_Radial_D5.0mm_P2.50mm
- C10, C6, C7, C9: footprint Capacitor_THT:CP_Radial_D4.0mm_P2.00mm -> Capacitor_THT:CP_Radial_D5.0mm_P2.50mm
- J5, J6: footprint Connector_IDC:IDC-Header_2x03_P2.54mm_Horizontal -> Connector_PinHeader_2.54mm:PinHeader_2x03_P2.54mm_Horizontal
Connections:
- net +5V: now also TP5.1
- net +VDC: now also TP2.1
- net -5V: now also TP3.1
- net -VDC: now also TP1.1
- net lm317_vi: now also D1.1 (K), D15.1 (K)
- net lm337_vi: now also D13.2 (A), D16.2 (A)
- net puente_in: now also D1.2 (A), D13.1 (K)
- net puente_in2: now also D15.2 (A), D16.1 (K)
