File: kicad_diseño/fuente_simetrica_24v/alimentacion.kicad_sch (KiCad schematic)
At the start: 54 parts, among them J1 Entrada +-24V, J2 5V_salida, J3 Salida +-24V, J5 Conn_02x03_Odd_Even, J6 Conn_02x03_Odd_Even, K1 SANYOU_SRD_Form_C, K2 SANYOU_SRD_Form_C, Q1 BC548, Q2 BC548, U1 LM317_TO-220, U2 LM337_TO220, U3 LM7805_TO220, U4 PC817, U5 PC817, U9 LM7905_TO220

Commit message: Update Fte - Diseño pcb
Parts:
- F1: footprint (none) -> Fuse:Fuseholder_Clip-5x20mm_Littelfuse_100_Inline_P20.50x4.60mm_D1.30mm_Horizontal
Connections:
- net GND: now also R7.1; no longer J2.2 (Pin_2), J3.2 (Pin_2), J6.3 (Pin_3), R7.2
- net V1_shunt renamed GND1
- net GND1: now also J2.2 (Pin_2), J3.2 (Pin_2), R7.2; no longer R7.1
- no-connect marks 2 -> 3
Other:
- moved on the sheet: R7
