File: kicad_diseño/fuente_simetrica_24v/_autosave-alimentacion.kicad_sch (KiCad schematic)
At the start: 54 parts, among them J1 Entrada +-24V, J2 5V_salida, J3 Salida +-24V, J5 Conn_02x03_Odd_Even, J6 Conn_02x03_Odd_Even, K1 SANYOU_SRD_Form_C, K2 SANYOU_SRD_Form_C, Q1 BC548, Q2 BC548, U1 LM317_TO-220, U2 LM337_TO220, U3 LM7805_TO220, U4 PC817, U5 PC817, U9 LM7905_TO220

Commit message: Update Fte - Diseño ao
Connections:
- net GND: no longer J6.3 (Pin_3)
- no-connect marks 2 -> 3
Changed lines of the file:
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@@
-	)
-	(junction
-		(at 152.4 52.07)
-		(diameter 0)
-		(color 0 0 0 0)
 	)
 	(junction
@@
 		(at 80.01 102.87)
 	)
+	(no_connect
+		(at 172.72 133.35)
+	)
 	(wire
 		(pts
@@
 	(wire
 		(pts
-			(xy 158.75 52.07) (xy 152.4 52.07)
-		)
-		(stroke
-			(width 0)
-			(type default)
-		)
-	)
-	(wire
-		(pts
 			(xy 196.85 34.29) (xy 204.47 34.29)
 		)
@@
 		(pts
 			(xy 102.87 46.99) (xy 104.14 46.99)
-		)
-		(stroke
-			(width 0)
-			(type default)
-		)
-	)
-	(wire
-		(pts
-			(xy 158.75 53.34) (xy 158.75 52.07)
 		)
 		(stroke
@@
 		)
 	)
-	(label "V2_shunt"
-		(at 172.72 133.35 180)
-		(fields_autoplaced yes)
-		(effects
-			(font
-				(size 1.27 1.27)
-				(bold yes)
-				(italic yes)
-			)
-			(justify right bottom)
-		)
-	)
 	(label "puente_in"
 		(at 38.1 44.45 0)
@@
 		)
 	)
-	(label "V2_shunt"
-		(at 158.75 53.34 270)
-		(fields_autoplaced yes)
-		(effects
-			(font
-				(size 1.27 1.27)
-				(bold yes)
-				(italic yes)
-			)
-			(justify right bottom)
-		)
-	)
