File: kicad_diseño/fuente_simetrica_24v/_autosave-control.kicad_sch (KiCad schematic)
At the start: 32 parts, among them J4 Comunicacion, J7 Conn_02x03_Odd_Even, J8 Conn_02x03_Odd_Even, Q3 BC548, SW1 BOOT, SW2 RESET, SW3 RotaryEncoder_Switch, U10 LM358, U6 ESP32-WROOM-32E, U7 AMS1117-3.3, U8 TL082

Commit message: Update Fte - Diseño ao
Connections:
- net V2_shunt: no longer names the net of J8.3 (Pin_3)
- no-connect marks 6 -> 7
Changed lines of the file:
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@@
+	)
+	(no_connect
+		(at 220.98 29.21)
 	)
 	(no_connect
@@
 			)
 			(justify right bottom)
-		)
-	)
-	(label "V2_shunt"
-		(at 220.98 29.21 180)
-		(fields_autoplaced yes)
-		(effects
-			(font
-				(size 1.27 1.27)
-				(bold yes)
-				(italic yes)
-			)
-			(justify right bottom)
