File: kicad_diseño/fuente_simetrica_24v/fuente_simetrica_24v.kicad_pcb (KiCad board)
At the start: 2 copper layers, 150 x 150 mm, 74 parts, among them J1 Entrada +-24V, J2 5V_salida, J3 Screw_Terminal_01x03, J4 Conn_01x04_Socket, K1 SANYOU_SRD_Form_C, K2 SANYOU_SRD_Form_C, Q1 BC548, Q2 BC548, Q3 BC548, SW1 SW_Push, SW2 SW_Push, SW3 RotaryEncoder_Switch, U1 LM317_TO-220, U10 LM358, U2 LM337_TO220, U3 LM7805_TO220, U4 PC817, U5 PC817, U6 ESP32-WROOM-32E, U7 AMS1117-3.3, U8 LM358, U9 LM7905_TO220

Commit message: Update Fte
Parts:
- R18: footprint LED_THT:LED_D5.0mm -> Resistor_THT:R_Axial_DIN0207_L6.3mm_D2.5mm_P10.16mm_Horizontal
- RV3: footprint Connector_PinHeader_2.54mm:PinHeader_1x03_P2.54mm_Vertical -> Connector_PinSocket_2.54mm:PinSocket_1x03_P2.54mm_Vertical
- RV4: footprint Connector_PinHeader_2.54mm:PinHeader_1x03_P2.54mm_Vertical -> Potentiometer_THT:Potentiometer_Bourns_3296W_Vertical
- U6, U7: moved to B.Cu
- moved U10 266.5 mm to (132.0, 91.4)
- moved D14 262.7 mm to (164.2, 93.3), turned to 90 degrees
- moved R18 262.3 mm to (149.0, 84.4), turned to -90 degrees
- moved R17 253.4 mm to (156.2, 108.5), turned to 90 degrees
- moved R16 246.0 mm to (149.0, 98.2), turned to -90 degrees
- moved Q3 237.4 mm to (123.4, 110.5)
- moved RV5 235.2 mm to (157.2, 92.4), turned to -90 degrees
- moved J2 226.4 mm to (165.0, 57.8), turned to 90 degrees
- moved R9 221.9 mm to (117.2, 130.3), turned to 180 degrees
- moved R12 219.8 mm to (117.2, 126.0), turned to 180 degrees
- moved BZ1 218.0 mm to (128.0, 123.0), turned to -90 degrees
- moved R15 207.4 mm to (108.8, 114.0)
- moved R19 206.0 mm to (108.9, 109.0)
- moved R7 197.5 mm to (155.6, 69.5), turned to 180 degrees
- moved J4 164.4 mm to (57.5, 140.0), turned to 90 degrees
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Other:
- board size 150 x 150 mm -> 150 x 130 mm

Commit message: Update Fte
Parts:
- removed D12, D13: D_Zener, Diode_THT:D_DO-35_SOD27_P7.62mm_Horizontal
- removed R13, R14, R8: R, Resistor_THT:R_Axial_DIN0207_L6.3mm_D2.5mm_P10.16mm_Horizontal
- removed RV2: R_Potentiometer_Trim, Potentiometer_THT:Potentiometer_Bourns_3296W_Vertical
- removed U8: LM358, Package_DIP:DIP-8_W7.62mm_LongPads
- added D10: D_Zener, Diode_THT:D_DO-35_SOD27_P7.62mm_Horizontal, F.Cu at (-14.0, 33.1)
- added D11: D_Zener, Diode_THT:D_DO-35_SOD27_P7.62mm_Horizontal, F.Cu at (-14.0, 36.6)
- added J5: Conn_02x03_Odd_Even, Connector_IDC:IDC-Header_2x03_P2.54mm_Horizontal, F.Cu at (-48.7, 56.3)
- added J6: Conn_02x03_Odd_Even, Connector_IDC:IDC-Header_2x03_P2.54mm_Horizontal, F.Cu at (-31.5, 56.3)
- added J7: Conn_02x03_Odd_Even, Connector_IDC:IDC-Header_2x03_P2.54mm_Horizontal, F.Cu at (-35.4, 20.1)
- added J8: Conn_02x03_Odd_Even, Connector_IDC:IDC-Header_2x03_P2.54mm_Horizontal, F.Cu at (-18.2, 20.1)
- added R20: 50k, Resistor_THT:R_Axial_DIN0207_L6.3mm_D2.5mm_P10.16mm_Horizontal, F.Cu at (-50.1, 16.0)
- added R21: 50k, Resistor_THT:R_Axial_DIN0207_L6.3mm_D2.5mm_P10.16mm_Horizontal, F.Cu at (-50.1, 20.1)
- added R22: 25k, Resistor_THT:R_Axial_DIN0207_L6.3mm_D2.5mm_P10.16mm_Horizontal, F.Cu at (-50.1, 24.1)
- added R23: 25k, Resistor_THT:R_Axial_DIN0207_L6.3mm_D2.5mm_P10.16mm_Horizontal, F.Cu at (-50.1, 28.1)
- added R24: 25k, Resistor_THT:R_Axial_DIN0207_L6.3mm_D2.5mm_P10.16mm_Horizontal, F.Cu at (-50.1, 32.2)
- added R25: 25k, Resistor_THT:R_Axial_DIN0207_L6.3mm_D2.5mm_P10.16mm_Horizontal, F.Cu at (-50.1, 36.2)
- added R26: 10k, Resistor_THT:R_Axial_DIN0207_L6.3mm_D2.5mm_P10.16mm_Horizontal, F.Cu at (-50.1, 40.3)
- added RV6: RG, Potentiometer_THT:Potentiometer_Bourns_3296W_Vertical, F.Cu at (-18.6, 34.5)
- added RV7: 10k, Potentiometer_THT:Potentiometer_Bourns_3296W_Vertical, F.Cu at (-18.6, 41.0)
- added TP1: lm337_out, TestPoint:TestPoint_2Pads_Pitch5.08mm_Drill1.3mm, F.Cu at (61.9, 87.0)
- added TP2: lm7805_out, TestPoint:TestPoint_2Pads_Pitch5.08mm_Drill1.3mm, F.Cu at (61.9, 91.7)
- added TP3: lm7905_out, TestPoint:TestPoint_2Pads_Pitch5.08mm_Drill1.3mm, F.Cu at (61.9, 96.3)
- added TP4: lm337_out, TestPoint:TestPoint_2Pads_Pitch5.08mm_Drill1.3mm, F.Cu at (61.9, 101.0)
- added U11: LM324, Package_DIP:DIP-12_W7.62mm_LongPads, F.Cu at (-36.4, 33.4)
- C3, C4: value 2000uF -> 2200uF
- J3: value Screw_Terminal_01x03 -> Salida +-24V
- J4: value Conn_01x04_Socket -> Comunicacion
- R16, R18: value R -> 68k
- R17: value R -> 10k
- RV1: value 10k -> 5k
- RV3: value 10k -> 5k; footprint Connector_PinSocket_2.54mm:PinSocket_1x03_P2.54mm_Vertical -> Connector_PinHeader_2.54mm:PinHeader_1x03_P2.54mm_Vertical
- RV5: value R_Potentiometer_Trim -> 10k
- SW1: value SW_Push -> BOOT
- SW2: value SW_Push -> RESET
- moved U7 182.6 mm to (-124.7, 99.8)
- moved C13 170.7 mm to (-128.3, 119.6)
- moved SW1 170.7 mm to (-21.9, 119.3)
- moved BZ1 170.7 mm to (-42.7, 124.8)
- moved C14 170.7 mm to (-133.7, 119.5)
- moved D14 170.7 mm to (-6.50, 95.2)
- moved DS1 170.7 mm to (-87.1, 140.5)
- moved J4 170.7 mm to (-113.2, 141.8)
- moved Q3 170.7 mm to (-47.3, 112.3)
- moved R12 170.7 mm to (-53.5, 127.8)
- moved R15 170.7 mm to (-61.9, 115.8)
- moved R16 170.7 mm to (-21.7, 100.1)
- moved R17 170.7 mm to (-14.5, 110.3)
- moved R18 170.7 mm to (-21.7, 86.2)
- moved R19 170.7 mm to (-61.8, 110.8)
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Connections:
- net Net-(D1-+) renamed /alimentacion/lm317_vi
- net Net-(D1--) renamed /alimentacion/lm337_vi
- net Net-(J1-Pin_1) renamed /alimentacion/puente_in
- net Net-(J1-Pin_3) renamed /alimentacion/puente_in2
- net Net-(J3-Pin_1) renamed /alimentacion/rele 1
- net Net-(J3-Pin_3) renamed /alimentacion/rele 2
- net Vshunt renamed /alimentacion/V1_shunt
- BZ1 pad 2: GND -> GND2
- C10 pad 2: Net-(D6-K) -> /alimentacion/lm337_vadj
- C13 pad 2: GND -> GND2
- C14 pad 2: GND -> GND2
- C9 pad 1: Net-(D5-A) -> /alimentacion/lm317_vadj
- D14 pad 2: GND -> GND2
- D5 pad 2: Net-(D5-A) -> /alimentacion/lm317_vadj
- D6 pad 1: Net-(D6-K) -> /alimentacion/lm337_vadj
- DS1 pad 1: GND -> GND2
- DS1 pad 16: GND -> GND2
- DS1 pad 5: GND -> GND2
- J4 pad 4: GND -> GND2
- R1 pad 2: Net-(U1-ADJ) -> /alimentacion/lm317_vadj
- R16 pad 1: Net-(R16-Pad1) -> /control/-24V
- R16 pad 2: Net-(U10A--) -> Net-(R16-Pad2)
- R17 pad 1: Net-(U10A--) -> Net-(R16-Pad2)
- R17 pad 2: /control/IO35 -> Net-(U10B--)
- R18 pad 1: -VDC -> /control/+24V
- R18 pad 2: Net-(R16-Pad1) -> Net-(U10A-+)
- R2 pad 1: Net-(U2-ADJ) -> /alimentacion/lm337_vadj
- RV1 pad 2: Net-(U2-ADJ) -> /alimentacion/lm337_vadj
- RV1 pad 3: Net-(U2-ADJ) -> /alimentacion/lm337_vadj
- RV3 pad 1: Net-(U1-ADJ) -> /alimentacion/lm317_vadj
- RV3 pad 2: Net-(U1-ADJ) -> /alimentacion/lm317_vadj
- RV4 pad 3: GND -> GND2
- RV5 pad 1: Net-(R16-Pad1) -> Net-(U10A-+)
- RV5 pad 2: GND -> GND2
- RV5 pad 3: GND -> GND2
- SW1 pad 2: GND -> GND2
- SW2 pad 1: GND -> GND2
- SW3 pad C: GND -> GND2
- SW3 pad S2: GND -> GND2
- U1 pad 1: Net-(U1-ADJ) -> /alimentacion/lm317_vadj
- U10 pad 2: Net-(U10A--) -> /control/IO35
- U10 pad 3: GND -> Net-(U10A-+)
- U10 pad 5: (no net) -> GND2
- U10 pad 6: (no net) -> Net-(U10B--)
- U10 pad 7: (no net) -> /control/IO15
- U2 pad 1: Net-(U2-ADJ) -> /alimentacion/lm337_vadj
- U4 pad 1: RELE_POSITIVO -> /alimentacion/RELE 1
- U5 pad 1: RELE_NEGATIVO -> /alimentacion/RELE 2
- U6 pad 1: GND -> GND2
- U6 pad 14: RELE_POSITIVO -> /control/IO12
- U6 pad 15: GND -> GND2
- U6 pad 16: RELE_POSITIVO -> /control/IO13
- U6 pad 38: GND -> GND2
- U6 pad 39: GND -> GND2
- U7 pad 1: GND -> GND2
Routing:
- net /alimentacion/puente_in: track 0.00 -> 59.5 mm
- net /alimentacion/lm317_vi: track 0.00 -> 51.3 mm
- net /alimentacion/lm337_vi: track 0.00 -> 40.6 mm
- net /alimentacion/puente_in2: track 0.00 -> 20.8 mm
Other:
- board size 150 x 130 mm -> 150 x 71 mm

Commit message: Update Fte - Diseño de Pcb
Parts:
- moved TP4 68.7 mm to (104.5, 47.0)
- moved TP2 51.1 mm to (105.5, 65.0)
- moved TP1 45.1 mm to (75.5, 44.0)
- moved TP3 31.9 mm to (76.5, 68.0)
- moved RV3 20.5 mm to (73.9, 23.0), turned to 90 degrees
- moved RV1 14.9 mm to (87.0, 23.0), turned to 90 degrees
- moved R2 1.75 mm to (109.0, 42.4)
- moved Q2 1.21 mm to (114.0, 30.7)
Routing:
- net +5V: track 0.00 -> 143.3 mm
- net -VDC: track 0.00 -> 100.5 mm
- net /alimentacion/lm317_vadj: track 0.00 -> 71.6 mm, vias 0 -> 2
- net /alimentacion/lm337_vadj: track 0.00 -> 62.8 mm
- net /alimentacion/lm337_vi: track 40.6 -> 86.4 mm
- net +VDC: track 0.00 -> 45.2 mm, vias 0 -> 2
- net Net-(D9-A): track 0.00 -> 39.7 mm
- net /alimentacion/lm317_vi: track 51.3 -> 88.4 mm
- net Net-(D7-A): track 0.00 -> 36.3 mm
- net /alimentacion/rele 1: track 0.00 -> 27.2 mm
- net /alimentacion/rele 2: track 0.00 -> 21.8 mm
- net Net-(R5-Pad1): track 0.00 -> 16.7 mm
- net Net-(R4-Pad1): track 0.00 -> 15.5 mm
- net Net-(Q2-B): track 0.00 -> 14.5 mm
- net -5V: track 0.00 -> 14.2 mm
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
Commit message: Update Fte - Fte Potencia
Parts:
- removed TP4: lm337_out, TestPoint:TestPoint_2Pads_Pitch5.08mm_Drill1.3mm
- added D13: 1N5407, Diode_THT:D_DO-201AD_P15.24mm_Horizontal, F.Cu at (33.6, 71.8)
- added D15: 1N5407, Diode_THT:D_DO-201AD_P15.24mm_Horizontal, F.Cu at (33.6, 78.5)
- added D16: 1N5407, Diode_THT:D_DO-201AD_P15.24mm_Horizontal, F.Cu at (33.4, 85.2)
- added REF**: MountingHole_3.2mm_M3, MountingHole:MountingHole_3.2mm_M3, F.Cu at (164.0, 94.0)
- added REF**: MountingHole_3.2mm_M3, MountingHole:MountingHole_3.2mm_M3, F.Cu at (26.0, 94.0)
- added REF**: MountingHole_3.2mm_M3, MountingHole:MountingHole_3.2mm_M3, F.Cu at (26.0, 26.0)
- added REF**: MountingHole_3.2mm_M3, MountingHole:MountingHole_3.2mm_M3, F.Cu at (164.0, 26.0)
- added TP5: lm7805_out, TestPoint:TestPoint_Pad_D3.0mm, F.Cu at (110.2, 77.0)
- C1, C11, C12, C2, C5, C8: footprint Capacitor_THT:CP_Radial_D4.0mm_P1.50mm -> Capacitor_THT:CP_Radial_D5.0mm_P2.50mm
- C10, C6, C7, C9: footprint Capacitor_THT:CP_Radial_D4.0mm_P2.00mm -> Capacitor_THT:CP_Radial_D5.0mm_P2.50mm
- D1: value W01G -> 1N5407; footprint Diode_THT:Diode_Bridge_Round_D9.8mm -> Diode_THT:D_DO-201AD_P15.24mm_Horizontal
- J5, J6: footprint Connector_IDC:IDC-Header_2x03_P2.54mm_Horizontal -> Connector_PinHeader_2.54mm:PinHeader_2x03_P2.54mm_Horizontal
- TP1, TP3: footprint TestPoint:TestPoint_2Pads_Pitch5.08mm_Drill1.3mm -> TestPoint:TestPoint_Pad_D3.0mm
- TP2: value lm7805_out -> lm317_out; footprint TestPoint:TestPoint_2Pads_Pitch5.08mm_Drill1.3mm -> TestPoint:TestPoint_Pad_D3.0mm
- moved J5 121.1 mm to (66.5, 93.3), turned to -90 degrees
- moved J6 115.1 mm to (77.5, 93.2), turned to -90 degrees
- moved J2 40.1 mm to (147.9, 94.0), turned to 0 degrees
- moved TP1 34.7 mm to (110.2, 44.5)
- moved TP2 32.9 mm to (79.7, 44.5)
- moved R10 26.7 mm to (139.1, 87.0), turned to 180 degrees
- moved R5 22.1 mm to (139.2, 26.0), turned to 180 degrees
- moved R4 19.6 mm to (139.1, 82.0), turned to 180 degrees
- moved J3 16.9 mm to (165.0, 62.0)
- moved D8 16.7 mm to (106.9, 92.9)
- moved R2 16.4 mm to (108.9, 26.0), turned to 0 degrees
- moved R3 13.5 mm to (87.9, 93.0)
- moved C8 11.7 mm to (101.8, 84.0)
- moved U3 11.7 mm to (97.2, 77.0)
- moved C7 11.5 mm to (94.7, 84.0)
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Connections:
- D1 pad 2: /alimentacion/puente_in2 -> /alimentacion/puente_in
- TP1 pad 1: +VDC -> -VDC
- TP2 pad 1: +5V -> +VDC
Routing:
- net +5V: track 143.3 -> 0.00 mm
- net -VDC: track 100.5 -> 0.00 mm
- net /alimentacion/lm317_vi: track 88.4 -> 0.00 mm
- net /alimentacion/lm337_vi: track 86.4 -> 0.00 mm
- net /alimentacion/lm317_vadj: track 71.6 -> 0.00 mm, vias 2 -> 0
- net /alimentacion/lm337_vadj: track 62.8 -> 0.00 mm
- net /alimentacion/puente_in: track 59.5 -> 0.00 mm
- net +VDC: track 45.2 -> 0.00 mm, vias 2 -> 0
- net Net-(D9-A): track 39.7 -> 0.00 mm
- net Net-(D7-A): track 36.3 -> 0.00 mm
- net /alimentacion/rele 1: track 27.2 -> 0.00 mm
- net /alimentacion/rele 2: track 21.8 -> 0.00 mm
- net /alimentacion/puente_in2: track 20.8 -> 0.00 mm
- net Net-(R5-Pad1): track 16.7 -> 0.00 mm
- net Net-(R4-Pad1): track 15.5 -> 0.00 mm
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Other:
- board size 150 x 71 mm -> 150 x 80 mm
- board text added: "Pote LM317"
- board text added: "Pote LM337"

Commit message: Update Fte - Control
Parts:
- added REF**: MountingHole_3.2mm_M3, MountingHole:MountingHole_3.2mm_M3, F.Cu at (164.0, 124.0)
- added REF**: MountingHole_3.2mm_M3, MountingHole:MountingHole_3.2mm_M3, F.Cu at (26.0, 177.0)
- added REF**: MountingHole_3.2mm_M3, MountingHole:MountingHole_3.2mm_M3, F.Cu at (164.0, 177.0)
- added REF**: MountingHole_3.2mm_M3, MountingHole:MountingHole_3.2mm_M3, F.Cu at (26.0, 124.0)
- J7, J8: footprint Connector_IDC:IDC-Header_2x03_P2.54mm_Horizontal -> Connector_PinSocket_2.54mm:PinSocket_2x03_P2.54mm_Horizontal
- moved U7 291.2 mm to (160.7, 157.8)
- moved U6 220.7 mm to (137.5, 159.0)
- moved R6 191.0 mm to (45.0, 202.0)
- moved D14 186.7 mm to (139.6, 211.4)
- moved R17 186.7 mm to (131.6, 226.5)
- moved RV5 186.7 mm to (132.6, 210.4)
- moved R16 186.7 mm to (124.4, 216.3)
- moved R18 186.7 mm to (124.4, 202.4)
- moved R20 185.6 mm to (-1.00, 195.0)
- moved R21 185.6 mm to (-1.00, 199.1)
- moved R22 185.6 mm to (-1.00, 203.1)
- moved R23 185.6 mm to (-1.00, 207.2)
- moved R24 185.6 mm to (-1.00, 211.2)
- moved R25 185.6 mm to (-1.00, 215.2)
- moved R26 185.6 mm to (-1.00, 219.3)
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Other:
- board size 150 x 80 mm -> 150 x 163 mm

Commit message: Update Fte - Diseño pcb
Parts:
- added F1: Fuse, Fuse:Fuseholder_Clip-5x20mm_Littelfuse_100_Inline_P20.50x4.60mm_D1.30mm_Horizontal, F.Cu at (26.0, 59.8)
- added R8: R, Resistor_THT:R_Axial_DIN0207_L6.3mm_D2.5mm_P10.16mm_Horizontal, F.Cu at (192.4, 122.0)
- added REF**: MountingHole_3.5mm_Pad, MountingHole:MountingHole_3.5mm_Pad, F.Cu at (40.0, 25.0)
- added REF**: MountingHole_3.5mm_Pad, MountingHole:MountingHole_3.5mm_Pad, F.Cu at (152.0, 25.0)
- added RV2: 10k, Potentiometer_THT:Potentiometer_Bourns_3296W_Vertical, F.Cu at (199.0, 139.0)
- added U8: TL082, Package_DIP:DIP-8_W7.62mm_LongPads, F.Cu at (192.8, 126.1)
- D10: value D_Zener -> 3.3V
- moved J5 110.7 mm to (163.0, 39.0), turned to 0 degrees
- moved J6 95.0 mm to (163.0, 52.0), turned to 0 degrees
- moved J3 88.4 mm to (81.8, 92.0), turned to 0 degrees
- moved R7 83.3 mm to (72.6, 78.5)
- moved J2 80.0 mm to (67.9, 92.0)
- moved U9 77.7 mm to (130.0, 33.0)
- moved TP3 75.0 mm to (143.8, 38.0)
- moved C11 74.4 mm to (127.5, 46.0)
- moved C12 74.4 mm to (134.5, 46.0)
- moved R5 53.8 mm to (152.5, 78.1), turned to 90 degrees
- moved D8 49.9 mm to (57.0, 93.0), turned to 180 degrees
- moved R10 46.6 mm to (95.0, 72.0), turned to 90 degrees
- moved D16 46.3 mm to (37.2, 39.1), turned to -90 degrees
- moved R11 46.1 mm to (157.0, 68.0), turned to -90 degrees
- moved U3 44.8 mm to (105.5, 32.9)
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Connections:
- C1 pad 2: GND -> GND1
- C10 pad 1: GND -> GND1
- C2 pad 2: GND -> GND1
- C3 pad 2: GND -> GND1
- C4 pad 1: GND -> GND1
- C5 pad 1: GND -> GND1
- C6 pad 1: GND -> GND1
- C9 pad 2: GND -> GND1
- J1 pad 1: /alimentacion/puente_in -> Net-(J1-Pin_1)
- J2 pad 2: GND -> GND1
- J3 pad 2: /alimentacion/V1_shunt -> GND1
- J6 pad 1: /alimentacion/V1_shunt -> GND1
- J6 pad 3: GND -> unconnected-(J6-Pin_3-Pad3)
- J8 pad 3: /control/V2_shunt -> unconnected-(J8-Pin_3-Pad3)
- R7 pad 2: /alimentacion/V1_shunt -> GND1
- RV1 pad 1: GND -> GND1
- RV3 pad 3: GND -> GND1
Routing:
- net +5V: track 0.00 -> 268.6 mm, vias 0 -> 2
- net +VDC: track 0.00 -> 227.8 mm, vias 0 -> 6
- net -VDC: track 0.00 -> 219.1 mm, vias 0 -> 2
- net /alimentacion/lm317_vi: track 0.00 -> 210.8 mm, vias 0 -> 2
- net /alimentacion/lm337_vi: track 0.00 -> 196.4 mm
- net GND: track 0.00 -> 132.6 mm, vias 0 -> 12
- net Net-(D9-A): track 0.00 -> 71.6 mm
- net /alimentacion/RELE 1: track 0.00 -> 63.2 mm, vias 0 -> 4
- net /alimentacion/rele 2: track 0.00 -> 44.0 mm
- net /alimentacion/RELE 2: track 0.00 -> 43.4 mm, vias 0 -> 2
- net /alimentacion/puente_in: track 0.00 -> 42.5 mm
- net -5V: track 0.00 -> 41.3 mm
- net /alimentacion/lm337_vadj: track 0.00 -> 39.5 mm, vias 0 -> 2
- net /alimentacion/lm317_vadj: track 0.00 -> 37.1 mm
- net Net-(R10-Pad1): track 0.00 -> 36.5 mm, vias 0 -> 2
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- added copper zone on B.Cu, net GND
- added copper zone on B.Cu, net GND1
